Commit message: docs(nav_bot_description): update table format and adjust sensor positions
update README.md table layout for better readability
adjust lidar and camera mounting positions in properties.xacro

File: src/nav_bot_description/urdf/common/properties.xacro (robot description, xacro)
@@ -65,5 +65,5 @@
   <xacro:property name="lidar_height"      value="0.065"/>
   <xacro:property name="lidar_mass"        value="0.19"/>
-  <xacro:property name="lidar_xyz"         value="${[0.16, 0.0, 0.28]}"/>  <!-- 收进顶板投影内，坐于顶板上方 -->
+  <xacro:property name="lidar_xyz"         value="${[0.13, 0.0, 0.28]}"/>  <!-- 收进顶板投影内，坐于顶板上方 -->
   <!-- IMU 36×24×10 mm，0.02 kg，贴近轮轴、刚性固定，周边 100 mm 内禁止动力线 -->
   <xacro:property name="imu_x"             value="0.036"/>
@@ -89,5 +89,5 @@
   <xacro:property name="camera_size"       value="0.038"/>
   <xacro:property name="camera_mass"       value="0.05"/>
-  <xacro:property name="camera_xyz"        value="${[0.195, 0.10, 0.0]}"/>  <!-- 相对 platform_link，骑前缘半嵌 -->
+  <xacro:property name="camera_xyz"        value="${[0.235, 0.0, -0.04]}"/>  <!-- 相对 platform_link，骑前缘半嵌 -->
   <xacro:property name="camera_pitch"      value="0.0"/>
   <!-- 前脸灯带（纯视觉件，参考整机渲染风格）：底盘前面板细长条 -->

Commit message: docs: 更新机器人模型参数与传感器描述
调整轮半径为0.09m，同步更新相关文档说明
修改相机与深度相机的安装描述，明确安装位置细节
调整IMU的Z轴安装偏移量以匹配实际硬件配置

File: src/nav_bot_description/urdf/common/properties.xacro (robot description, xacro)
@@ -15,6 +15,6 @@
 -->
 <robot xmlns:xacro="http://www.ros.org/wiki/xacro">
-  <!-- ======================== 运动学基准（R = 0.10 m） ======================== -->
-  <xacro:property name="wheel_radius"      value="0.10"/>   <!-- 轮半径 Ø200 mm -->
+  <!-- ======================== 运动学基准（R = 0.09 m） ======================== -->
+  <xacro:property name="wheel_radius"      value="0.09"/>   <!-- 轮半径 Ø180 mm -->
   <xacro:property name="wheel_width"       value="0.060"/>  <!-- 轮宽 60 mm -->
   <xacro:property name="track_width"       value="0.48"/>   <!-- 轮距：左右轮 y = ±0.24 -->
@@ -71,5 +71,5 @@
   <xacro:property name="imu_z"             value="0.010"/>
   <xacro:property name="imu_mass"          value="0.02"/>
-  <xacro:property name="imu_xyz"           value="${[0.0, 0.0, 0.02]}"/>
+  <xacro:property name="imu_xyz"           value="${[0.0, 0.0, 0.06]}"/>
   <!-- 深度相机 90×25×25 mm，0.07 kg
        外形 v2.4（隐藏式）：link 水平、完全藏进车头（y=0 正中），前脸唯一可见部分是

File: src/nav_bot_description/urdf/nav_bot.urdf.xacro (robot description, xacro)
@@ -8,8 +8,8 @@
     ├── platform_link                      fixed
     │   ├── arm_base_link                  fixed（机械臂预留基座）
-    │   └── camera_link                    fixed（RGB 摄像头 + 短支架）
+    │   └── camera_link                    fixed（RGB 摄像头，平嵌顶板前缘）
     ├── lidar_link                         fixed（平台前部，扫描面离地 0.28 m）
     ├── imu_link                           fixed（底盘中心贴轮轴）
-    └── depth_camera_link                  fixed（前面板俯仰 -15°）
+    └── depth_camera_link                  fixed（前面板隐藏式，-15° 下俯在 Gazebo 传感器 pose）
   用法：
     xacro src/nav_bot_description/urdf/nav_bot.urdf.xacro > nav_bot.urdf

File: src/nav_bot_description/urdf/wheels.xacro (robot description, xacro)
@@ -3,5 +3,5 @@
   wheels.xacro — 四轮独立驱动（4WD 差速）：lf / rf / lb / rb，全部 continuous 绕 y 轴
   规范（robot_params.yaml v2.0）：轮安装点 x=±0.26（轴距 0.52）、y=±0.24（轮距 0.48）、
-  z=R=0.10；同侧两轮速度指令一致；轮地摩擦 mu ≥ 0.9（见 gazebo.xacro）。
+  z=R=0.09；同侧两轮速度指令一致；轮地摩擦 mu ≥ 0.9（见 gazebo.xacro）。
   视觉件含朝向车体的短轮轴，避免轮子与车身之间出现悬空缝隙。
 -->
