Commit message: docs: 更新URDF材质注释并替换底盘颜色为白色

File: src/nav_bot_description/urdf/base.xacro (robot description, xacro)
@@ -12,5 +12,5 @@
         <cylinder radius="${column_radius}" length="${column_height}"/>
       </geometry>
-      <material name="chassis_dark"/>
+      <material name="body_white"/>
     </visual>
   </xacro:macro>
@@ -22,5 +22,5 @@
         <box size="${chassis_x} ${chassis_y} ${chassis_z}"/>
       </geometry>
-      <material name="chassis_dark"/>
+      <material name="body_white"/>
     </visual>
     <!-- 前脸灯带：底盘前面板细长青色灯条（纯视觉件，参考整机渲染风格） -->

File: src/nav_bot_description/urdf/common/materials.xacro (robot description, xacro)
@@ -6,5 +6,5 @@
 -->
 <robot xmlns:xacro="http://www.ros.org/wiki/xacro">
-  <!-- 机身主色 #E8ECF1（顶板/外壳） -->
+  <!-- 车身主色 白色 #E8ECF1（底盘箱体/顶板/角柱） -->
   <material name="body_white">
     <color rgba="${0xE8/255.0} ${0xEC/255.0} ${0xF1/255.0} 1.0"/>

Commit message: docs: 更新 nav_bot_description 至外观 v2.5，替换基础几何体为网格模型

File: src/nav_bot_description/urdf/base.xacro (robot description, xacro)
@@ -5,30 +5,15 @@
 -->
 <robot xmlns:xacro="http://www.ros.org/wiki/xacro">
-  <!-- 顶板角柱视觉件（在 platform_link 坐标系中：柱底 = 底盘顶面，柱顶 = 顶板底面） -->
-  <xacro:macro name="platform_column" params="x y">
-    <visual>
-      <origin xyz="${x} ${y} ${-(platform_z / 2.0 + column_height / 2.0)}" rpy="0 0 0"/>
-      <geometry>
-        <cylinder radius="${column_radius}" length="${column_height}"/>
-      </geometry>
-      <material name="body_white"/>
-    </visual>
-  </xacro:macro>
+  <!-- 外观网格（外观 v2.5）：visual 引用 meshes/ 下的 .dae（自带材质色）；
+       碰撞体保持简化几何体（规范要求，禁止复用外观 mesh）。 -->
   <!-- ==================== base_link 底盘框架 520×400×120 mm ==================== -->
   <link name="base_link">
+    <!-- 外观 mesh：底盘箱体 + 前脸青色灯带（已在 mesh 内合并，坐标以 link 原点为基准） -->
     <visual>
-      <origin xyz="0 0 ${chassis_center_z}" rpy="0 0 0"/>
+      <origin xyz="0 0 0" rpy="0 0 0"/>
       <geometry>
-        <box size="${chassis_x} ${chassis_y} ${chassis_z}"/>
+        <mesh filename="package://nav_bot_description/meshes/base_link.dae"/>
       </geometry>
-      <material name="body_white"/>
-    </visual>
-    <!-- 前脸灯带：底盘前面板细长青色灯条（纯视觉件，参考整机渲染风格） -->
-    <visual>
-      <origin xyz="${chassis_x / 2.0} 0 ${front_strip_cz}" rpy="0 0 0"/>
-      <geometry>
-        <box size="${front_strip_y} ${front_strip_x} ${front_strip_z}"/>
-      </geometry>
-      <material name="accent_cyan"/>
+      <material name="chassis_dark"/>
     </visual>
     <collision>
@@ -58,16 +43,12 @@
   </joint>
   <link name="platform_link">
+    <!-- 外观 mesh：顶板 + 四根支撑角柱（已在 mesh 内合并） -->
     <visual>
       <origin xyz="0 0 0" rpy="0 0 0"/>
       <geometry>
-        <box size="${platform_x} ${platform_y} ${platform_z}"/>
+        <mesh filename="package://nav_bot_description/meshes/platform_link.dae"/>
       </geometry>
       <material name="body_white"/>
     </visual>
-    <!-- 四角支撑立柱：底盘顶面 -> 顶板底面（视觉件，消除顶板悬空感） -->
-    <xacro:platform_column x="${column_xy[0]}"  y="${column_xy[1]}"/>
-    <xacro:platform_column x="${column_xy[0]}"  y="${-column_xy[1]}"/>
-    <xacro:platform_column x="${-column_xy[0]}" y="${column_xy[1]}"/>
-    <xacro:platform_column x="${-column_xy[0]}" y="${-column_xy[1]}"/>
     <collision>
       <origin xyz="0 0 0" rpy="0 0 0"/>
@@ -87,8 +68,7 @@
   <link name="arm_base_link">
     <visual>
-      <!-- 板上表面与关节面齐平：中心抬高半厚 -->
-      <origin xyz="0 0 ${arm_base_z / 2.0}" rpy="0 0 0"/>
+      <origin xyz="0 0 0" rpy="0 0 0"/>
       <geometry>
-        <box size="${arm_base_x} ${arm_base_y} ${arm_base_z}"/>
+        <mesh filename="package://nav_bot_description/meshes/arm_base_link.dae"/>
       </geometry>
       <material name="accent_amber"/>

File: src/nav_bot_description/urdf/sensors.xacro (robot description, xacro)
@@ -18,16 +18,9 @@
   </joint>
   <link name="lidar_link">
+    <!-- 外观 mesh：雷达筒 + 底座法兰（已在 mesh 内合并） -->
     <visual>
       <origin xyz="0 0 0" rpy="0 0 0"/>
       <geometry>
-        <cylinder radius="${lidar_radius}" length="${lidar_height}"/>
-      </geometry>
-      <material name="sensor_navy"/>
-    </visual>
-    <!-- 底座法兰：桥接顶板面与雷达筒底，无外伸杆件 -->
-    <visual>
-      <origin xyz="0 0 ${lidar_flange_z}" rpy="0 0 0"/>
-      <geometry>
-        <cylinder radius="${lidar_flange_radius}" length="0.012"/>
+        <mesh filename="package://nav_bot_description/meshes/lidar_link.dae"/>
       </geometry>
       <material name="sensor_navy"/>
@@ -51,5 +44,5 @@
       <origin xyz="0 0 0" rpy="0 0 0"/>
       <geometry>
-        <box size="${imu_x} ${imu_y} ${imu_z}"/>
+        <mesh filename="package://nav_bot_description/meshes/imu_link.dae"/>
       </geometry>
       <material name="sensor_navy"/>
@@ -72,9 +65,9 @@
   </joint>
   <link name="depth_camera_link">
-    <!-- 玻璃视窗：与前面板齐平的深色镜面小窗（唯一可见部分） -->
+    <!-- 外观 mesh：前脸齐平玻璃视窗（唯一可见部分，机身藏于车头内无外观） -->
     <visual>
-      <origin xyz="0.0015 0 0" rpy="0 0 0"/>
+      <origin xyz="0 0 0" rpy="0 0 0"/>
       <geometry>
-        <box size="0.003 ${depth_cam_win_y} ${depth_cam_win_z}"/>
+        <mesh filename="package://nav_bot_description/meshes/depth_camera_link.dae"/>
       </geometry>
       <material name="lens_dark"/>
@@ -106,18 +99,11 @@
   </joint>
   <link name="camera_link">
+    <!-- 外观 mesh：相机方块 + 前侧镜头圆片（已在 mesh 内合并） -->
     <visual>
       <origin xyz="0 0 0" rpy="0 0 0"/>
       <geometry>
-        <box size="${camera_size} ${camera_size} ${camera_size}"/>
+        <mesh filename="package://nav_bot_description/meshes/camera_link.dae"/>
       </geometry>
       <material name="camera_gray"/>
-    </visual>
-    <!-- 镜头面：前侧小圆片，增加辨识度（纯视觉件） -->
-    <visual>
-      <origin xyz="${camera_size / 2.0 + 0.001} 0 0" rpy="0 ${pi/2.0} 0"/>
-      <geometry>
-        <cylinder radius="${0.55 * camera_size / 2.0}" length="0.002"/>
-      </geometry>
-      <material name="tire_black"/>
     </visual>
     <collision>

File: src/nav_bot_description/urdf/wheels.xacro (robot description, xacro)
@@ -19,19 +19,11 @@
     </joint>
     <link name="wheel_${name}_link">
+      <!-- 外观 mesh：轮胎 + 朝车体侧的短轮轴（已在 mesh 内合并，四轮共用） -->
       <visual>
-        <!-- URDF 圆柱轴沿 z，绕 x 转 90° 使轮轴对齐 y -->
-        <origin xyz="0 0 0" rpy="${pi/2.0} 0 0"/>
+        <origin xyz="0 0 0" rpy="0 0 0"/>
         <geometry>
-          <cylinder radius="${wheel_radius}" length="${wheel_width}"/>
+          <mesh filename="package://nav_bot_description/meshes/wheel.dae"/>
         </geometry>
         <material name="tire_black"/>
-      </visual>
-      <!-- 轮轴：朝车体一侧伸出的短轴（视觉件） -->
-      <visual>
-        <origin xyz="0 ${-y_sign * axle_length / 2.0} 0" rpy="${pi/2.0} 0 0"/>
-        <geometry>
-          <cylinder radius="${axle_radius}" length="${axle_length}"/>
-        </geometry>
-        <material name="sensor_navy"/>
       </visual>
       <collision>

Commit message: fix: 将网格模型从DAE改为STL以解决Gazebo渲染纯白问题
注释说明Gazebo 8.15的ColladaLoader无法解析DAE颜色材质，因此将所有URDF中的mesh引用从.dae文件改为.stl文件，并添加experiments目录到.gitignore，删除空的.gitkeep文件。

File: src/nav_bot_description/urdf/base.xacro (robot description, xacro)
@@ -13,5 +13,5 @@
       <origin xyz="0 0 0" rpy="0 0 0"/>
       <geometry>
-        <mesh filename="package://nav_bot_description/meshes/base_link.dae"/>
+        <mesh filename="package://nav_bot_description/meshes/base_link.stl"/>
       </geometry>
       <material name="chassis_dark"/>
@@ -47,5 +47,5 @@
       <origin xyz="0 0 0" rpy="0 0 0"/>
       <geometry>
-        <mesh filename="package://nav_bot_description/meshes/platform_link.dae"/>
+        <mesh filename="package://nav_bot_description/meshes/platform_link.stl"/>
       </geometry>
       <material name="body_white"/>
@@ -70,5 +70,5 @@
       <origin xyz="0 0 0" rpy="0 0 0"/>
       <geometry>
-        <mesh filename="package://nav_bot_description/meshes/arm_base_link.dae"/>
+        <mesh filename="package://nav_bot_description/meshes/arm_base_link.stl"/>
       </geometry>
       <material name="accent_amber"/>

File: src/nav_bot_description/urdf/sensors.xacro (robot description, xacro)
@@ -22,5 +22,5 @@
       <origin xyz="0 0 0" rpy="0 0 0"/>
       <geometry>
-        <mesh filename="package://nav_bot_description/meshes/lidar_link.dae"/>
+        <mesh filename="package://nav_bot_description/meshes/lidar_link.stl"/>
       </geometry>
       <material name="sensor_navy"/>
@@ -44,5 +44,5 @@
       <origin xyz="0 0 0" rpy="0 0 0"/>
       <geometry>
-        <mesh filename="package://nav_bot_description/meshes/imu_link.dae"/>
+        <mesh filename="package://nav_bot_description/meshes/imu_link.stl"/>
       </geometry>
       <material name="sensor_navy"/>
@@ -69,5 +69,5 @@
       <origin xyz="0 0 0" rpy="0 0 0"/>
       <geometry>
-        <mesh filename="package://nav_bot_description/meshes/depth_camera_link.dae"/>
+        <mesh filename="package://nav_bot_description/meshes/depth_camera_link.stl"/>
       </geometry>
       <material name="lens_dark"/>
@@ -103,5 +103,5 @@
       <origin xyz="0 0 0" rpy="0 0 0"/>
       <geometry>
-        <mesh filename="package://nav_bot_description/meshes/camera_link.dae"/>
+        <mesh filename="package://nav_bot_description/meshes/camera_link.stl"/>
       </geometry>
       <material name="camera_gray"/>

File: src/nav_bot_description/urdf/wheels.xacro (robot description, xacro)
@@ -23,5 +23,5 @@
         <origin xyz="0 0 0" rpy="0 0 0"/>
         <geometry>
-          <mesh filename="package://nav_bot_description/meshes/wheel.dae"/>
+          <mesh filename="package://nav_bot_description/meshes/wheel.stl"/>
         </geometry>
         <material name="tire_black"/>

Commit message: refactor(nav_bot_description): 添加零质量base_footprint消除KDL惯性警告
新增base_footprint作为URDF根link，解决KDL报错
更新所有相关配置的TF帧和说明文档，确保坐标链正确

File: src/nav_bot_description/urdf/base.xacro (robot description, xacro)
@@ -7,4 +7,17 @@
   <!-- 外观网格（外观 v2.5）：visual 引用 meshes/ 下的 .dae（自带材质色）；
        碰撞体保持简化几何体（规范要求，禁止复用外观 mesh）。 -->
+  <!-- ==================== base_footprint（零质量根 link，仅用于 TF） ==================== -->
+  <!-- KDL（robot_state_publisher / RViz 的解析器）不支持根 link 带惯性，会刷
+       "The root link base_link has an inertia specified in the URDF" 警告。
+       这里加一个无质量的 base_footprint 作为根，与 base_link 固定且原点重合：
+         TF：odom -> base_footprint -> base_link -> 各传感器 link
+       Gazebo 侧固定关节会把 base_link 合并进 base_footprint（位姿/惯量不变），
+       所以 DiffDrive 的 child_frame_id 与 EKF 的 base_link_frame 都要写 base_footprint。 -->
+  <link name="base_footprint"/>
+  <joint name="base_footprint_joint" type="fixed">
+    <parent link="base_footprint"/>
+    <child link="base_link"/>
+    <origin xyz="0 0 0" rpy="0 0 0"/>
+  </joint>
   <!-- ==================== base_link 底盘框架 520×400×120 mm ==================== -->
   <link name="base_link">

File: src/nav_bot_description/urdf/common/properties.xacro (robot description, xacro)
@@ -6,5 +6,6 @@
   坐标系：REP-103（x 前 / y 左 / z 上）
   基准约定：base_link 原点在地面上（轮心 z = 轮半径 R），
-           即 base_link 同时承担 base_footprint 的角色，odom -> base_link 直接可用。
+           URDF 根 link 是零质量的 base_footprint（与 base_link 原点重合，见 base.xacro），
+           用于消除 KDL 的 "root link has an inertia" 警告：odom -> base_footprint -> base_link。
   外形修正（延续 4WD 版外形审查结论）：
     - 底盘宽 500 → 400 mm：轮距 y=±0.24 的四轮完全外露于车体两侧（420×500 稿

File: src/nav_bot_description/urdf/gazebo.xacro (robot description, xacro)
@@ -15,9 +15,13 @@
       <!-- ★ TF 改发到 /tf_gz_odom 且不做桥接。
            轮式里程计的 TF 在 4WD 滑移转向下误差极大（实测旋转虚报 2.6×），
-           odom->base_link 改由 robot_localization EKF 发布（见 config/ekf.yaml）。
+           odom->base_footprint 改由 robot_localization EKF 发布（见 config/ekf.yaml）。
            同一时刻只能有一个发布者，否则 TF 打架、odom 抽搐。 -->
       <tf_topic>/tf_gz_odom</tf_topic>
       <frame_id>odom</frame_id>
-      <child_frame_id>base_link</child_frame_id>
+      <!-- ★ 必须写 base_footprint：URDF 根 link 是零质量的 base_footprint，
+           base_link 通过固定关节挂在它下面，gz 合并后模型基准 link 就是 base_footprint。
+           写 base_link 会和 robot_state_publisher 发的 base_footprint->base_link
+           形成"一个子帧两个父帧"，TF 打架。 -->
+      <child_frame_id>base_footprint</child_frame_id>
       <min_linear_velocity>-${max_linear_vel}</min_linear_velocity>
       <max_linear_velocity>${max_linear_vel}</max_linear_velocity>

File: src/nav_bot_description/urdf/nav_bot.urdf.xacro (robot description, xacro)
@@ -3,13 +3,14 @@
   nav_bot.urdf.xacro — 顶层装配文件
   依据《轮式机器人建模规范》+ robot_params.yaml v2.0
-  拓扑：11 links / 10 joints
-    base_link（根，原点位于地面）
-    ├── wheel_lf/rf/lb/rb_link             continuous ×4（4WD 差速，同侧同速）
-    ├── platform_link                      fixed
-    │   ├── arm_base_link                  fixed（机械臂预留基座）
-    │   └── camera_link                    fixed（RGB 摄像头，平嵌顶板前缘）
-    ├── lidar_link                         fixed（平台前部，扫描面离地 0.28 m）
-    ├── imu_link                           fixed（底盘中心贴轮轴）
-    └── depth_camera_link                  fixed（前面板隐藏式，-15° 下俯在 Gazebo 传感器 pose）
+  拓扑：12 links / 11 joints
+    base_footprint（根，零质量，仅提供 TF）
+    └── base_link（原点位于地面）
+        ├── wheel_lf/rf/lb/rb_link             continuous ×4（4WD 差速，同侧同速）
+        ├── platform_link                      fixed
+        │   ├── arm_base_link                  fixed（机械臂预留基座）
+        │   └── camera_link                    fixed（RGB 摄像头，平嵌顶板前缘）
+        ├── lidar_link                         fixed（平台前部，扫描面离地 0.28 m）
+        ├── imu_link                           fixed（底盘中心贴轮轴）
+        └── depth_camera_link                  fixed（前面板隐藏式，-15° 下俯在 Gazebo 传感器 pose）
   用法：
     xacro src/nav_bot_description/urdf/nav_bot.urdf.xacro > nav_bot.urdf
